Commit message: update urdf and yaml

File: urdf/holiday_panda.urdf (robot description, URDF)
Before this commit: robot panda, 14 links, 13 joints
Links:
- removed link panda_link0
- removed link panda_link1
- removed link panda_link2
- removed link panda_link3
- removed link panda_link4
- removed link panda_link5
- removed link panda_link6
- removed link panda_link7
- removed link panda_link8
- added link ft_sensor_link; collision mesh filename=package://holiday_robot_descriptions/assets/object/collisio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 scale=0.001 0.001 0.001; visual mesh filename=package://holiday_robot_descriptions/assets/object/visual/a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 scale=0.001 0.001 0.001
- added link ft_sensor_mount_link; collision cylinder length=0.03 radius=0.04; visual cylinder length=0.03 radius=0.04
- added link hand_mount_link; collision cylinder length=0.025 radius=0.03; visual cylinder length=0.025 radius=0.03
- added link link0; collision mesh filename=../meshes/panda/link0.obj scale=1.0 1.0 1.0; visual mesh filename=../meshes/panda/link0.dae
- added link link1; collision mesh filename=../meshes/panda/link1.obj scale=1.0 1.0 1.0; visual mesh filename=../meshes/panda/link1.dae
- added link link2; collision mesh filename=../meshes/panda/link2.obj scale=1.0 1.0 1.0; visual mesh filename=../meshes/panda/link2.dae
- added link link3; collision mesh filename=../meshes/panda/link3.obj scale=1.0 1.0 1.0; visual mesh filename=../meshes/panda/link3.dae
- added link link4; collision mesh filename=../meshes/panda/link4.obj scale=1.0 1.0 1.0; visual mesh filename=../meshes/panda/link4.dae
- added link link5; collision mesh filename=../meshes/panda/link5.obj scale=1.0 1.0 1.0; visual mesh filename=../meshes/panda/link5.dae
- added link link6; collision mesh filename=../meshes/panda/link6.obj scale=1.0 1.0 1.0; visual mesh filename=../meshes/panda/link6.dae
- added link link7; collision mesh filename=../meshes/panda/link7.obj scale=1.0 1.0 1.0; visual mesh filename=../meshes/panda/link7.dae
- added link panda_fingertip_centered, mass 1.0e-6
- link panda_hand: geometry collision mesh filename=../meshes/panda/hand.obj; visual mesh filename=../meshes/panda/hand.dae
- link panda_leftfinger: geometry collision mesh filename=../meshes/panda/finger.obj; visual mesh filename=../meshes/panda/finger.dae
- link panda_rightfinger: geometry collision mesh filename=../meshes/panda/finger.obj; visual mesh filename=../meshes/panda/finger.dae
Joints:
- removed joint panda_joint1
- removed joint panda_joint2
- removed joint panda_joint3
- removed joint panda_joint4
- removed joint panda_joint5
- removed joint panda_joint6
- removed joint panda_joint7
- removed joint panda_joint8
- added joint ft_sensor_joint: type fixed, parent ft_sensor_mount_link, child ft_sensor_link, origin xyz=0 0 0.03 rpy=0 0 0
- added joint ft_sensor_mount_joint: type fixed, parent link7, child ft_sensor_mount_link, origin xyz=0 0 0.107 rpy=0 0 0.784602
- added joint hand_mount_joint: type fixed, parent ft_sensor_link, child hand_mount_link, origin xyz=0 0 0.02 rpy=0 0 0
- added joint joint1: type revolute, parent link0, child link1, origin xyz=0 0 0.333 rpy=0 0 0, axis 0 0 1, limit lower=-2.3093 upper=2.3093 effort=87 velocity=2.0
- added joint joint2: type revolute, parent link1, child link2, origin xyz=0 0 0 rpy=-1.57079632679 0 0, axis 0 0 1, limit lower=-1.5133 upper=1.5133 effort=87.0 velocity=1.0
- added joint joint3: type revolute, parent link2, child link3, origin xyz=0 -0.316 0 rpy=1.57079632679 0 0, axis 0 0 1, limit lower=-2.4937 upper=2.4937 effort=87.0 velocity=1.5
- added joint joint4: type revolute, parent link3, child link4, origin xyz=0.0825 0 0 rpy=1.57079632679 0 0, axis 0 0 1, limit lower=-2.7478 upper=-0.4461 effort=87.0 velocity=1.25
- added joint joint5: type revolute, parent link4, child link5, origin xyz=-0.0825 0.384 0 rpy=-1.57079632679 0 0, axis 0 0 1, limit lower=-2.48 upper=2.48 effort=12.0 velocity=3.0
- added joint joint6: type revolute, parent link5, child link6, origin xyz=0 0 0 rpy=1.57079632679 0 0, axis 0 0 1, limit lower=0.8521 upper=4.2094 effort=12.0 velocity=1.5
- added joint joint7: type revolute, parent link6, child link7, origin xyz=0.088 0 0 rpy=1.57079632679 0 0, axis 0 0 1, limit lower=-2.6895 upper=2.6895 effort=12.0 velocity=3.0
- added joint panda_fingertip_centered_joint: type fixed, parent panda_hand, child panda_fingertip_centered, origin xyz=0 0 0.1034 rpy=0 0 0
- joint panda_finger_joint1: limit lower=0.0 upper=0.04 effort=100 velocity=0.2 -> lower=0.0 upper=0.04 effort=20 velocity=0.2
- joint panda_finger_joint2: limit lower=0.0 upper=0.04 effort=100 velocity=0.2 -> lower=0.0 upper=0.04 effort=20 velocity=0.2; mimic joint=panda_finger_joint1 -> (none)
- joint panda_hand_joint: origin xyz=0 0 0 rpy=0 0 -0.7853981633974483 -> xyz=0 0 0.025 rpy=0 0 -1.5708; parent panda_link8 -> hand_mount_link
- joint panda_hand_tcp_joint: origin xyz=0 0 0.18 rpy=0 0 0 -> xyz=0 0 0.1034 rpy=0 0 0

Commit message: update README and config

File: urdf/holiday_panda.urdf (robot description, URDF)
Before this commit: robot fr3_gripper, 17 links, 16 joints
Links:
- removed link ft_sensor_link
- removed link ft_sensor_mount_link
- added link ft_sensor_and_mount_link; collision cylinder length=0.03 radius=0.04; visual cylinder length=0.03 radius=0.04
Joints:
- removed joint ft_sensor_joint
- removed joint ft_sensor_mount_joint
- added joint ft_sensor_and_mount_joint: type fixed, parent link7, child ft_sensor_and_mount_link, origin xyz=0 0 0.107 rpy=0 0 0.784602
- joint hand_mount_joint: origin xyz=0 0 0.02 rpy=0 0 0 -> xyz=0 0 0.05 rpy=0 0 0; parent ft_sensor_link -> ft_sensor_and_mount_link

Commit message: add friday

File: urdf/holiday_panda.urdf (robot description, URDF)
Before this commit: robot fr3_gripper, 16 links, 15 joints
Links:
- link ball_link: geometry visual sphere radius=0.01

File: urdf/holiday_xarm6.urdf (robot description, URDF)
Before this commit: robot xarm6, 8 links, 7 joints
Links:
- link ball_link: geometry visual sphere radius=0.01
