Commit message: add friday data

File: urdf/friday_left.urdf (robot description, URDF)
Before this commit: robot friday, 63 links, 62 joints
Links:
- removed link BASE
- removed link head_1
- removed link head_2
- removed link left_finger_1_1
- removed link left_finger_1_2
- removed link left_finger_1_3
- removed link left_finger_1_4
- removed link left_finger_2_1
- removed link left_finger_2_2
- removed link left_finger_2_3
- removed link left_finger_2_4
- removed link left_finger_3_1
- removed link left_finger_3_2
- removed link left_finger_3_3
- removed link left_finger_3_4
- removed link left_finger_4_1
- removed link left_finger_4_2
- removed link left_finger_4_3
- removed link left_finger_4_4
- removed link left_finger_5_1
- removed link left_finger_5_2
- removed link left_finger_5_3
- removed link left_finger_5_4
- removed link right_arm_1
- removed link right_arm_2
- removed link right_arm_3
- removed link right_arm_4
- removed link right_arm_5
- removed link right_arm_6
- removed link right_arm_7
- removed link right_finger_1_1
- removed link right_finger_1_2
- removed link right_finger_1_3
- removed link right_finger_1_4
- removed link right_finger_2_1
- removed link right_finger_2_2
- removed link right_finger_2_3
- removed link right_finger_2_4
- removed link right_finger_3_1
- removed link right_finger_3_2
- removed link right_finger_3_3
- removed link right_finger_3_4
- removed link right_finger_4_1
- removed link right_finger_4_2
- removed link right_finger_4_3
- removed link right_finger_4_4
- removed link right_finger_5_1
- removed link right_finger_5_2
- removed link right_finger_5_3
- removed link right_finger_5_4
- removed link waist_1
- removed link waist_2
- removed link waist_3
- removed link waist_4
Joints:
- removed joint head_1
- removed joint head_2
- removed joint left_finger_1_1
- removed joint left_finger_1_2
- removed joint left_finger_1_3
- removed joint left_finger_1_4
- removed joint left_finger_2_1
- removed joint left_finger_2_2
- removed joint left_finger_2_3
- removed joint left_finger_2_4
- removed joint left_finger_3_1
- removed joint left_finger_3_2
- removed joint left_finger_3_3
- removed joint left_finger_3_4
- removed joint left_finger_4_1
- removed joint left_finger_4_2
- removed joint left_finger_4_3
- removed joint left_finger_4_4
- removed joint left_finger_5_1
- removed joint left_finger_5_2
- removed joint left_finger_5_3
- removed joint left_finger_5_4
- removed joint right_arm_1
- removed joint right_arm_2
- removed joint right_arm_3
- removed joint right_arm_4
- removed joint right_arm_5
- removed joint right_arm_6
- removed joint right_arm_7
- removed joint right_finger_1_1
- removed joint right_finger_1_2
- removed joint right_finger_1_3
- removed joint right_finger_1_4
- removed joint right_finger_2_1
- removed joint right_finger_2_2
- removed joint right_finger_2_3
- removed joint right_finger_2_4
- removed joint right_finger_3_1
- removed joint right_finger_3_2
- removed joint right_finger_3_3
- removed joint right_finger_3_4
- removed joint right_finger_4_1
- removed joint right_finger_4_2
- removed joint right_finger_4_3
- removed joint right_finger_4_4
- removed joint right_finger_5_1
- removed joint right_finger_5_2
- removed joint right_finger_5_3
- removed joint right_finger_5_4
- removed joint waist_1
- removed joint waist_2
- removed joint waist_3
- removed joint waist_4
- removed joint waist_5

File: urdf/friday_right.urdf (robot description, URDF)
Before this commit: robot friday, 63 links, 62 joints
Links:
- removed link BASE
- removed link head_1
- removed link head_2
- removed link left_arm_1
- removed link left_arm_2
- removed link left_arm_3
- removed link left_arm_4
- removed link left_arm_5
- removed link left_arm_6
- removed link left_arm_7
- removed link left_finger_1_1
- removed link left_finger_1_2
- removed link left_finger_1_3
- removed link left_finger_1_4
- removed link left_finger_2_1
- removed link left_finger_2_2
- removed link left_finger_2_3
- removed link left_finger_2_4
- removed link left_finger_3_1
- removed link left_finger_3_2
- removed link left_finger_3_3
- removed link left_finger_3_4
- removed link left_finger_4_1
- removed link left_finger_4_2
- removed link left_finger_4_3
- removed link left_finger_4_4
- removed link left_finger_5_1
- removed link left_finger_5_2
- removed link left_finger_5_3
- removed link left_finger_5_4
- removed link right_finger_1_1
- removed link right_finger_1_2
- removed link right_finger_1_3
- removed link right_finger_1_4
- removed link right_finger_2_1
- removed link right_finger_2_2
- removed link right_finger_2_3
- removed link right_finger_2_4
- removed link right_finger_3_1
- removed link right_finger_3_2
- removed link right_finger_3_3
- removed link right_finger_3_4
- removed link right_finger_4_1
- removed link right_finger_4_2
- removed link right_finger_4_3
- removed link right_finger_4_4
- removed link right_finger_5_1
- removed link right_finger_5_2
- removed link right_finger_5_3
- removed link right_finger_5_4
- removed link waist_1
- removed link waist_2
- removed link waist_3
- removed link waist_4
Joints:
- removed joint head_1
- removed joint head_2
- removed joint left_arm_1
- removed joint left_arm_2
- removed joint left_arm_3
- removed joint left_arm_4
- removed joint left_arm_5
- removed joint left_arm_6
- removed joint left_arm_7
- removed joint left_finger_1_1
- removed joint left_finger_1_2
- removed joint left_finger_1_3
- removed joint left_finger_1_4
- removed joint left_finger_2_1
- removed joint left_finger_2_2
- removed joint left_finger_2_3
- removed joint left_finger_2_4
- removed joint left_finger_3_1
- removed joint left_finger_3_2
- removed joint left_finger_3_3
- removed joint left_finger_3_4
- removed joint left_finger_4_1
- removed joint left_finger_4_2
- removed joint left_finger_4_3
- removed joint left_finger_4_4
- removed joint left_finger_5_1
- removed joint left_finger_5_2
- removed joint left_finger_5_3
- removed joint left_finger_5_4
- removed joint right_finger_1_1
- removed joint right_finger_1_2
- removed joint right_finger_1_3
- removed joint right_finger_1_4
- removed joint right_finger_2_1
- removed joint right_finger_2_2
- removed joint right_finger_2_3
- removed joint right_finger_2_4
- removed joint right_finger_3_1
- removed joint right_finger_3_2
- removed joint right_finger_3_3
- removed joint right_finger_3_4
- removed joint right_finger_4_1
- removed joint right_finger_4_2
- removed joint right_finger_4_3
- removed joint right_finger_4_4
- removed joint right_finger_5_1
- removed joint right_finger_5_2
- removed joint right_finger_5_3
- removed joint right_finger_5_4
- removed joint waist_1
- removed joint waist_2
- removed joint waist_3
- removed joint waist_4
- removed joint waist_5
